Commit message: 2025.4.3

File: urdf/urdf/robot.urdf (robot description, URDF)
Before this commit: robot robot.SLDASM, 3 links, 2 joints
Links:
- removed link rob_link
- removed link wheel_Link
- added link rod_link, mass 0.24; collision mesh filename=package://robot/meshes/rod_link.STL; visual mesh filename=package://robot/meshes/rod_link.STL
- added link wheel_link, mass 0.47124; collision mesh filename=package://robot/meshes/wheel_link.STL; visual mesh filename=package://robot/meshes/wheel_link.STL
- link body_link: geometry collision mesh filename=package://robot/meshes/body_link.STL; visual mesh filename=package://robot/meshes/body_link.STL
Joints:
- removed joint rob_joint
- removed joint wheel_joint
- added joint body_rod_joint: type continuous, parent body_link, child rod_link, origin xyz=0 0 -0.115 rpy=0 0 0, axis -1 0 0
- added joint rod_wheel_joint: type continuous, parent rod_link, child wheel_link, origin xyz=0 0 -0.1 rpy=0 0 0, axis -1 0 0
